File: cad/bike/schematic/cadenza_rev_A/cadenza_rev_A.kicad_sch (KiCad schematic)
At the start: 36 parts, among them J1 USB_A, J2 USB_C_Receptacle, J3 Conn_01x02, Q1 BC547, U1 TLC5916, U10 HDSP-A151, U11 TLC5916, U12 HDSP-A151, U13 STM32F105RCTx, U14 INA193, U15 TLC5916, U2 HDSP-A151, U3 TLC5916, U4 HDSP-A151, U5 TLC5916, U6 HDSP-A151, U7 TLC5916, U8 HDSP-A151, U9 TLC5916

Commit message: new placement for the LED chips
Parts:
- added D9: LED, LED_THT:LED_D3.0mm, symbol Device:LED
Connections:
- net GND: now also D9.1 (K)
- net at U6.7 (DP): now also U5.12 (~{OUT7})
- net at U6.8 (C): now also U5.11 (~{OUT6})
- net at U6.9 (B): now also U5.10 (~{OUT5})
Other:
- note added: "Acceleration display"
- note added: "Unreliable estimation"

Commit message: routing progress update
Parts:
- added C3, C4, C5, C6: 100nF, Capacitor_SMD:C_0805_2012Metric_Pad1.18x1.45mm_HandSolder, symbol Device:C
- added R10, R8, R9: R_US, Resistor_SMD:R_0805_2012Metric_Pad1.20x1.40mm_HandSolder, symbol Device:R_US
Connections:
- net +3.3V: now also C3.2, C4.2, C5.2, C6.2
- net GND: now also C3.1, C4.1, C5.1, C6.1, R10.2, R8.2, R9.2
- net at U9.15 (R-EXT): now also R9.1
- net at U13.14 (PA0): now also U1.2 (SDI)
- net at U7.10 (~{OUT5}): now also U8.9 (B)
- net at U7.11 (~{OUT6}): now also U8.8 (C)
- net at U7.12 (~{OUT7}): now also U8.7 (DP)
- net at U7.15 (R-EXT): now also R8.1
- net at U7.5 (~{OUT0}): now also U8.5 (D)
- net at U7.6 (~{OUT1}): now also U8.4 (E)
- net at U7.7 (~{OUT2}): now also U8.3 (G)
- net at U7.8 (~{OUT3}): now also U8.2 (F)
- net at U7.9 (~{OUT4}): now also U8.10 (A)
- net at U11.15 (R-EXT): now also R10.1
- net at U6.10 (A): now also U5.9 (~{OUT4})
- net at U6.2 (F): now also U5.8 (~{OUT3})
- net at U6.3 (G): now also U5.7 (~{OUT2})
- net at U6.4 (E): now also U5.6 (~{OUT1})
- net at U6.5 (D): now also U5.5 (~{OUT0})
Other:
- moved on the sheet: R1, R2, U1, U10, U11, U2, U3, U4, U7, U8, U9

Commit message: switched to a new estimator
Connections:
- net at U9.11 (~{OUT6}): now also U10.8 (C)
- net at U9.12 (~{OUT7}): now also U10.7 (DP)
Other:
- moved on the sheet: R9, U10, U9

Commit message: routing progress update
Parts:
- added C7, C8: 100nF, Capacitor_SMD:C_0805_2012Metric_Pad1.18x1.45mm_HandSolder, symbol Device:C
Connections:
- net +3.3V: now also C7.2, C8.2
- net GND: now also C7.1, C8.1
- net at U9.10 (~{OUT5}): now also U10.9 (B)
- net at U9.5 (~{OUT0}): now also U10.5 (D)
- net at U9.6 (~{OUT1}): now also U10.4 (E)
- net at U9.7 (~{OUT2}): now also U10.3 (G)
- net at U9.8 (~{OUT3}): now also U10.2 (F)
- net at U9.9 (~{OUT4}): now also U10.10 (A)
- net at U11.10 (~{OUT5}): now also U12.9 (B)
- net at U11.11 (~{OUT6}): now also U12.8 (C)
- net at U11.12 (~{OUT7}): now also U12.7 (DP)
- net at U11.5 (~{OUT0}): now also U12.5 (D)
- net at U11.6 (~{OUT1}): now also U12.4 (E)
- net at U11.7 (~{OUT2}): now also U12.3 (G)
- net at U11.8 (~{OUT3}): now also U12.2 (F)
- net at U11.9 (~{OUT4}): now also U12.10 (A)
Other:
- moved on the sheet: C3, C4, C5, C6, D1, D2, D3, D4, D5, D6, D7, D8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

Commit message: added the SPI interface
Parts:
- added C10, C11, C9: 100nF, Capacitor_SMD:C_0805_2012Metric_Pad1.18x1.45mm_HandSolder, symbol Device:C
Connections:
- net +3.3V: now also C10.1, C11.1, C9.1
- net GND: now also C10.2, C11.2, C9.2
- net SPI_CLK: now reaches U1.3 (CLK), U11.3 (CLK), U15.3 (CLK), U3.3 (CLK), U5.3 (CLK), U7.3 (CLK), U9.3 (CLK)
- net SPI_CLK: now also U13.21 (PA5)
- net at U13.14 (PA0): no longer U1.2 (SDI)
- net SPI_MISO: now reaches U13.22 (PA6)
- net SPI_MISO: now also U15.14 (SDO)
- net SPI_MOSI: now reaches U13.23 (PA7)
- net SPI_MOSI: now also U1.2 (SDI)

Commit message: added routing for the acceleration LEDs
Parts:
- removed R7: 0.01, Resistor_SMD:R_1210_3225Metric_Pad1.30x2.65mm_HandSolder, symbol Device:R_US
- removed U14: INA193, Package_TO_SOT_SMD:SOT-23-5, symbol Amplifier_Current:INA193
- added J4: Conn_01x02, Connector_PinHeader_2.54mm:PinHeader_1x02_P2.54mm_Vertical, symbol Connector_Generic:Conn_01x02
Connections:
- net +3.3V: no longer C2.1
- net +5V: now also C2.1, J4.2 (Pin_2)
- net at J2.A4 (VBUS), J2.A9 (VBUS), J2.B4 (VBUS)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: now also J4.1 (Pin_1)
- net at D8.1 (K): now also U15.8 (~{OUT3}); no longer U15.12 (~{OUT7})
- net at U15.10 (~{OUT5}): now also D2.1 (K); no longer D6.1 (K)
- net at U15.11 (~{OUT6}): now also D3.1 (K); no longer D7.1 (K)
- net at U15.5 (~{OUT0}): now also D5.1 (K); no longer D1.1 (K)
- net at U15.6 (~{OUT1}): now also D6.1 (K); no longer D2.1 (K)
- net at U15.7 (~{OUT2}): now also D7.1 (K); no longer D3.1 (K)
- net at D4.1 (K): now also U15.12 (~{OUT7}); no longer U15.8 (~{OUT3})
- net at U15.9 (~{OUT4}): now also D1.1 (K); no longer D5.1 (K)
Other:
- moved on the sheet: C10, C11, C9

Commit message: routing progress update
Parts:
- added C12: 100nF, Capacitor_SMD:C_0805_2012Metric_Pad1.18x1.45mm_HandSolder, symbol Device:C
Connections:
- net +3.3V: now also C12.1
- net GND: now also C12.2
Changed lines of the file:
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@@
 	)
 	(junction
+		(at 339.09 71.12)
+		(diameter 0)
+		(color 0 0 0 0)
+	)
+	(junction
 		(at 78.74 81.28)
 		(diameter 0)
@@
 	(wire
 		(pts
+			(xy 353.06 71.12) (xy 339.09 71.12)
+		)
+		(stroke
+			(width 0)
+			(type default)
+		)
+	)
+	(wire
+		(pts
 			(xy 101.6 95.25) (xy 105.41 95.25)
 		)
@@
 	(wire
 		(pts
+			(xy 353.06 73.66) (xy 353.06 71.12)
+		)
+		(stroke
+			(width 0)
+			(type default)
+		)
+	)
+	(wire
+		(pts
 			(xy 171.45 78.74) (xy 218.44 78.74)
 		)
@@
 	(wire
 		(pts
+			(xy 353.06 81.28) (xy 353.06 83.82)
+		)
+		(stroke
+			(width 0)
+			(type default)
+		)
+	)
+	(wire
+		(pts
 			(xy 273.05 92.71) (xy 269.24 92.71)
 		)
@@
 	)
 	(symbol
+		(lib_id "power:GND")
+		(at 353.06 83.82 0)
+		(unit 1)
+		(body_style 1)
+		(exclude_from_sim no)
+		(in_bom yes)
+		(on_board yes)
+		(in_pos_files yes)
+		(dnp no)
+		(fields_autoplaced yes)
+		(property "Reference" "#PWR037"
+			(at 353.06 90.17 0)
+			(hide yes)
+			(show_name no)
+			(do_not_autoplace no)
+			(effects
+				(font
+					(size 1.27 1.27)
+				)
+			)
+		)
+		(property "Value" "GND"
+			(at 353.06 88.9 0)
+			(show_name no)
+			(do_not_autoplace no)
+			(effects
+				(font
+					(size 1.27 1.27)
+				)
+			)
+		)
+		(property "Footprint" ""
+			(at 353.06 83.82 0)
+			(hide yes)
+			(show_name no)
+			(do_not_autoplace no)
+			(effects
+				(font
+					(size 1.27 1.27)
+				)
+			)
+		)
+		(property "Datasheet" ""
+			(at 353.06 83.82 0)
+			(hide yes)
+			(show_name no)
+			(do_not_autoplace no)
+			(effects
+				(font
+					(size 1.27 1.27)
+				)
+			)
+		)
+		(property "Description" "Power symbol creates a global label with name \"GND\" , ground"
+			(at 353.06 83.82 0)
+			(hide yes)
+			(show_name no)
+			(do_not_autoplace no)
+			(effects
+				(font
+					(size 1.27 1.27)
+				)
+			)
+		)
+		(pin "1"
+		)
+		(instances
+			(project "cadenza_rev_A"
+				(path "/dbb6f7df-ddcf-4018-ba7f-ab9ccecd39f9"
+					(reference "#PWR037")
+					(unit 1)
+				)
+			)
+		)
+	)
+	(symbol
 		(lib_id "Display_Character:HDSP-A151")
 		(at 121.92 54.61 0)
@@
 					(unit 1)
 				)
+			)
+		)
+	)
+	(symbol
+		(lib_id "Device:C")
+		(at 353.06 77.47 0)
+		(unit 1)
+		(body_style 1)
+		(exclude_from_sim no)
+		(in_bom yes)
+		(on_board yes)
+		(in_pos_files yes)
+		(dnp no)
+		(fields_autoplaced yes)
+		(property "Reference" "C12"
+			(at 356.87 76.1999 0)
+			(show_name no)
+			(do_not_autoplace no)
+			(effects
+				(font
+					(size 1.27 1.27)
+				)
+				(justify left)
+			)
+		)
+		(property "Value" "100nF"
+			(at 356.87 78.7399 0)
+			(show_name no)
+			(do_not_autoplace no)
+			(effects
+				(font
+					(size 1.27 1.27)
+				)
+				(justify left)
+			)
+		)
+		(property "Footprint" "Capacitor_SMD:C_0805_2012Metric_Pad1.18x1.45mm_HandSolder"
+			(at 354.0252 81.28 0)
+			(hide yes)
+			(show_name no)
+			(do_not_autoplace no)
+			(effects
+				(font
+					(size 1.27 1.27)
+				)
+			)
+		)
+		(property "Datasheet" ""
+			(at 353.06 77.47 0)
+			(hide yes)
+			(show_name no)
+			(do_not_autoplace no)
+			(effects
+				(font
+					(size 1.27 1.27)
+				)
+			)
+		)
+		(property "Description" "Unpolarized capacitor"
+			(at 353.06 77.47 0)
+			(hide yes)
+			(show_name no)
+			(do_not_autoplace no)
+			(effects
+				(font
+					(size 1.27 1.27)
+				)
+			)
+		)
+		(pin "1"
+		)
+		(pin "2"
+		)
+		(instances
+			(project "cadenza_rev_A"
+				(path "/dbb6f7df-ddcf-4018-ba7f-ab9ccecd39f9"
+					(reference "C12")
+					(unit 1)
+				)
